File: stepper_card/stepper_card.kicad_pcb (KiCad board)
At the start: 2 copper layers, 53.6 x 68 mm, 25 parts, among them J1 Bus_PCI_Express_x1, J2 Conn_01x04, J3 Conn_01x06_Pin, J4 Conn_01x01_Pin, J5 Conn_01x01_Pin, J6 Conn_01x01_Pin, J7 Conn_01x01_Pin, J8 Conn_01x01_Pin, SW1 SW_DIP_x04, U1 DRV8825PWPR_Stepper_Driver

Commit message: changed pinout
Connections:
- J1 pad A11: unconnected-(J1-PadA11) -> +3V3
- J1 pad A12: +3V3 -> VM
- J1 pad A3: /CIPO -> /SCLK
- J1 pad A5: /SCLK -> /CIPO
- J1 pad B11: unconnected-(J1-PadB11) -> +3V3
- J1 pad B12: +3V3 -> VM
- J3 pad 2: /CIPO -> /SCLK
- J3 pad 4: /SCLK -> /CIPO
Routing:
- net +3V3: track 126.4 -> 130.7 mm
- net /SCLK: track 57.5 -> 61.6 mm
- net /CIPO: track 61.6 -> 57.5 mm
- net VM: track 115.3 -> 115.8 mm
- added copper zone on B.Cu, net VM

Commit message: changed pinout and added pullup onto cs
Parts:
- added R4: 10k, Resistor_SMD:R_0201_0603Metric_Pad0.64x0.40mm_HandSolder, F.Cu at (137.5, 104.0)
- moved J5 3.76 mm to (138.0, 101.5)
- moved J6 3.76 mm to (138.0, 96.5)
Connections:
- J1 pad A1: /STEP -> /SCL
- J1 pad A10: Net-(J1-PadA10) -> unconnected-(J1-PadA10)
- J1 pad A2: /DIR -> /SDA
- J1 pad A3: /SCLK -> /CS
- J1 pad A4: /COPI -> /CIPO
- J1 pad A5: /CIPO -> /COPI
- J1 pad A6: /CS -> /SCLK
- J1 pad A7: /SDA -> /STEP
- J1 pad A8: /SCL -> /DIR
- J1 pad A9: Net-(J1-PadA10) -> unconnected-(J1-PadA9)
- J1 pad B1: /nFAULT -> unconnected-(J1-PadB1)
- J1 pad B8: unconnected-(J1-PadB8) -> /nFAULT
- J3 pad 2: /SCLK -> /CS
- J3 pad 3: /COPI -> /CIPO
- J3 pad 4: /CIPO -> /COPI
- J3 pad 5: /CS -> /SCLK
Routing:
- net /CS: track 55.5 -> 63.2 mm
- net /SCLK: track 61.6 -> 55.5 mm
- net /nFAULT: track 45.8 -> 50.4 mm
- net /COPI: track 59.6 -> 57.5 mm
- net /CIPO: track 57.5 -> 59.6 mm
- net /DIR: track 52.9 -> 51.5 mm
- net Net-(J1-PadA10): track 1.00 -> 0.00 mm
- net (no net): track 0.00 -> 1.00 mm
- net +3V3: track 130.7 -> 131.7 mm
- net /STEP: track 52.4 -> 53.2 mm
