File: stepper_card/stepper_card.kicad_sch (KiCad schematic)
At the start: 25 parts, among them J1 Bus_PCI_Express_x1, J2 Conn_01x04, J3 Conn_01x06_Pin, J4 Conn_01x01_Pin, J5 Conn_01x01_Pin, J6 Conn_01x01_Pin, J7 Conn_01x01_Pin, J8 Conn_01x01_Pin, SW1 SW_DIP_x04, U1 DRV8825PWPR_Stepper_Driver

Commit message: changed pinout and added pullup onto cs
Parts:
- added R4: 10k, Resistor_SMD:R_0201_0603Metric_Pad0.64x0.40mm_HandSolder, symbol Device:R
Connections:
- net +3V3: now also R4.1
- net CIPO: now also J1.A4, J3.3 (Pin_3); no longer J1.A5, J3.4 (Pin_4)
- net COPI: now also J1.A5, J3.4 (Pin_4); no longer J1.A4, J3.3 (Pin_3)
- net CS: now also J1.A3, J3.2 (Pin_2), R4.2; no longer J1.A6, J3.5 (Pin_5)
- net DIR: now also J1.A8; no longer J1.A2
- net SCL: now also J1.A1; no longer J1.A8
- net SCLK: now also J1.A6, J3.5 (Pin_5); no longer J1.A3, J3.2 (Pin_2)
- net SDA: now also J1.A2; no longer J1.A7
- net STEP: now also J1.A7; no longer J1.A1
- net nFAULT: now also J1.B8; no longer J1.B1
- net at J1.A10: no longer J1.A9
Other:
- moved on the sheet: C1, C2, C3, C4, C5, C6, J1A, J1B, J2, R1, R2, R3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
